Commit message: change link length
Change-Id: Ie5481c3a1a2ca12820be8d650acb821caa845352

File: urdf/mini_cheetah_urdf.urdf (robot description, URDF)
Before this commit: robot mini_cheetah, 17 links, 16 joints
Joints:
- joint abduct_fl_to_thigh_fl_j: origin xyz=0.0 0.062 0.00 rpy=0.0 0.0 0.0 -> xyz=0.0 0.067 0.00 rpy=0.0 0.0 0.0
- joint abduct_fr_to_thigh_fr_j: origin xyz=0.0 -0.062 0.00 rpy=0.0 0.0 0.0 -> xyz=0.0 -0.067 0.00 rpy=0.0 0.0 0.0
- joint abduct_hl_to_thigh_hl_j: origin xyz=0.0 0.062 0.00 rpy=0.0 0.0 0.0 -> xyz=0.0 0.067 0.00 rpy=0.0 0.0 0.0
- joint abduct_hr_to_thigh_hr_j: origin xyz=0.0 -0.062 0.00 rpy=0.0 0.0 0.0 -> xyz=0.0 -0.067 0.00 rpy=0.0 0.0 0.0
