Commit message: 1
Change-Id: I8665ae9223d59046af9f04521e1bf28d891735b9

File: urdf/quadruped_robot.urdf (robot description, URDF)
Before this commit: robot mini_cheetah, 17 links, 16 joints
Links:
- link abduct_fl: mass 0.54 -> 0.517
- link abduct_fr: mass 0.54 -> 0.517
- link abduct_hl: mass 0.54 -> 0.517
- link abduct_hr: mass 0.54 -> 0.517
- link body: mass 3.3 -> 4.267
- link thigh_fl: mass 0.634 -> 0.729
- link thigh_fr: mass 0.634 -> 0.729
- link thigh_hl: mass 0.634 -> 0.729
- link thigh_hr: mass 0.634 -> 0.729
- link toe_fl: geometry collision sphere radius=0.020; visual sphere radius=0.020
- link toe_fr: geometry collision sphere radius=0.020; visual sphere radius=0.020
- link toe_hl: geometry collision sphere radius=0.020; visual sphere radius=0.020
- link toe_hr: geometry collision sphere radius=0.020; visual sphere radius=0.020
Joints:
- joint abduct_fl_to_thigh_fl_j: origin xyz=0.0 0.067 0.00 rpy=0.0 0.0 0.0 -> xyz=0.0 0.0671 0.00 rpy=0.0 0.0 0.0
- joint abduct_fr_to_thigh_fr_j: origin xyz=0.0 -0.067 0.00 rpy=0.0 0.0 0.0 -> xyz=0.0 -0.0671 0.00 rpy=0.0 0.0 0.0
- joint abduct_hl_to_thigh_hl_j: origin xyz=0.0 0.067 0.00 rpy=0.0 0.0 0.0 -> xyz=0.0 0.0671 0.00 rpy=0.0 0.0 0.0
- joint abduct_hr_to_thigh_hr_j: origin xyz=0.0 -0.067 0.00 rpy=0.0 0.0 0.0 -> xyz=0.0 -0.0671 0.00 rpy=0.0 0.0 0.0
- joint thigh_fl_to_knee_fl_j: origin xyz=0.0 0.0 -0.209 rpy=0.0 0 0.0 -> xyz=0.0 0.0 -0.206 rpy=0.0 0 0.0
- joint thigh_fr_to_knee_fr_j: origin xyz=0.0 0.0 -0.209 rpy=0.0 0 0.0 -> xyz=0.0 0.0 -0.206 rpy=0.0 0 0.0
- joint thigh_hl_to_knee_hl_j: origin xyz=0.0 0.0 -0.209 rpy=0.0 0 0.0 -> xyz=0.0 0.0 -0.206 rpy=0.0 0 0.0
- joint thigh_hr_to_knee_hr_j: origin xyz=0.0 0.0 -0.209 rpy=0.0 0 0.0 -> xyz=0.0 0.0 -0.206 rpy=0.0 0 0.0
- joint toe_fl_joint: origin xyz=0 0 -0.18 -> xyz=0 0 -0.185
- joint toe_fr_joint: origin xyz=0 0 -0.18 -> xyz=0 0 -0.185
- joint toe_hl_joint: origin xyz=0 0 -0.18 -> xyz=0 0 -0.185
- joint toe_hr_joint: origin xyz=0 0 -0.18 -> xyz=0 0 -0.185
